Commit message: Description: Fixed wheel and wheel joint orientations

File: drivebot_description/urdf/drivebot_model.xacro (robot description, xacro)
@@ -23,19 +23,23 @@
     <material>Gazebo/Orange</material>
   </gazebo>
-  <xacro:cylinderLink name="leftWheel" mass="${wheelMass}" r="${wheelR}" h="${wheelH}" color="red" />
+  <xacro:cylinderLink
+      name="leftWheel" mass="${wheelMass}" radius="${wheelR}" height="${wheelH}" color="red" p ="${pi/2}" />
   <joint name="leftWheel_joint" type="continuous">
     <parent link="body_link" />
     <child link="leftWheel_link" />
-    <origin xyz="${-bodyX/4} ${-bodyY/2 - wheelH/2} 0" rpy="${pi/2} 0 0" />
+    <origin xyz="${-bodyX/4} ${bodyY/2 + wheelH/2} 0" rpy="0 0 ${pi/2}" />
   </joint>
+  <xacro:jointTransmission name="leftWheel" />
   <gazebo reference="leftWheel_link">
     <material>Gazebo/Red</material>
   </gazebo>
-  <xacro:cylinderLink name="rightWheel" mass="${wheelMass}" r="${wheelR}" h="${wheelH}" color="green" />
+  <xacro:cylinderLink
+      name="rightWheel" mass="${wheelMass}" radius="${wheelR}" height="${wheelH}" color="green" p ="${pi/2}"/>
   <joint name="rightWheel_joint" type="continuous">
     <parent link="body_link" />
     <child link="rightWheel_link" />
-    <origin xyz="${-bodyX/4} ${bodyY/2 + wheelH/2} 0" rpy="${-pi/2} 0 0" />
+    <origin xyz="${-bodyX/4} ${-bodyY/2 - wheelH/2} 0" rpy="0 0 ${pi/2}" />
   </joint>
+  <xacro:jointTransmission name="rightWheel" />
   <gazebo reference="rightWheel_link">
     <material>Gazebo/Green</material>

File: drivebot_description/urdf/macros.xacro (robot description, xacro)
@@ -41,21 +41,21 @@
     </link>
   </xacro:macro>
-  <xacro:macro name="cylinderLink" params="name mass r h color:=grey">
+  <xacro:macro name="cylinderLink" params="name mass radius height r:=0 p:=0 y:=0 color:=grey">
     <link name="${name}_link">
       <inertia>
-        <origin xyz="0 0 0" rpy="0 0 0"/>
+        <origin xyz="0 0 0" rpy="${r} ${p} ${y}"/>
         <mass value="${mass}"/>
-        <xacro:cylinder_inertia mass="${mass}" r="${r}" h="${h}"/>
+        <xacro:cylinder_inertia mass="${mass}" r="${radius}" h="${height}"/>
       </inertia>
       <collision>
-        <origin xyz="0 0 0" rpy="0 0 0" />
+        <origin xyz="0 0 0" rpy="${r} ${p} ${y}"/>
         <geometry>
-          <cylinder radius="${r}" length="${h}"/>
+          <cylinder radius="${radius}" length="${height}"/>
         </geometry>
       </collision>
       <visual>
-        <origin xyz="0 0 0" rpy="0 0 0"/>
+        <origin xyz="0 0 0" rpy="${r} ${p} ${y}"/>
         <geometry>
-          <cylinder radius="${r}" length="${h}"/>
+          <cylinder radius="${radius}" length="${height}"/>
         </geometry>
         <material name="${color}"/>
@@ -85,11 +85,11 @@
     </link>
   </xacro:macro>
-  <xacro:macro name="joint_transmission" params="joint_name reduction:=10">
-    <transmission name="${joint_name}_transmission">
+  <xacro:macro name="jointTransmission" params="name reduction:=10">
+    <transmission name="${name}_transmission">
       <type>transmission_interface/SimpleTransmission</type>
-      <joint name="${joint_name}_joint">
+      <joint name="${name}_joint">
         <hardwareInterface>hardware_interface/EffortJointInterface</hardwareInterface>
       </joint>
-      <actuator name="${joint_name}_servo">
+      <actuator name="${name}_servo">
         <hardwareInterface>EffortJointInterface</hardwareInterface>
         <mechanicalReduction>${reduction}</mechanicalReduction>

Commit message: Fixed inertia typo and shrank caster wheel

File: drivebot_description/urdf/drivebot_model.xacro (robot description, xacro)
@@ -11,5 +11,5 @@
   <xacro:property name="wheelH" value="0.1" />
   <xacro:property name="wheelMass" value="1" />
-  <xacro:property name="casterR" value="${wheelR}" />
+  <xacro:property name="casterR" value="${(wheelR - bodyZ / 2) / 2}" />
   <xacro:property name="casterMass" value="${1}" />
   <link name="base_link" />
@@ -49,7 +49,7 @@
     <parent link="body_link" />
     <child link="caster_link" />
-    <origin xyz="${bodyX/4} 0 0" rpy="0 0 0" />
+    <origin xyz="${bodyX/4} 0 ${-(bodyZ/2 + casterR)}" rpy="0 0 0" />
   </joint>
-  <gazebo reference="rightWheel_link">
+  <gazebo reference="caster_link">
     <material>Gazebo/Black</material>
   </gazebo>

File: drivebot_description/urdf/macros.xacro (robot description, xacro)
@@ -21,9 +21,9 @@
   <xacro:macro name="boxLink" params="name mass x y z color:=grey">
     <link name="${name}_link">
-      <inertia>
+      <inertial>
         <origin xyz="0 0 0" rpy="0 0 0"/>
         <mass value="${mass}"/>
         <xacro:box_inertia mass="${mass}" x="${x}" y="${y}" z="${z}"/>
-      </inertia>
+      </inertial>
       <collision>
         <origin xyz="0 0 0" rpy="0 0 0" />
@@ -43,9 +43,9 @@
   <xacro:macro name="cylinderLink" params="name mass radius height r:=0 p:=0 y:=0 color:=grey">
     <link name="${name}_link">
-      <inertia>
+      <inertial>
         <origin xyz="0 0 0" rpy="${r} ${p} ${y}"/>
         <mass value="${mass}"/>
         <xacro:cylinder_inertia mass="${mass}" r="${radius}" h="${height}"/>
-      </inertia>
+      </inertial>
       <collision>
         <origin xyz="0 0 0" rpy="${r} ${p} ${y}"/>

Commit message: Description: Repaired model for Gazebo diff_drive simulation

File: drivebot_description/urdf/drivebot_model.xacro (robot description, xacro)
@@ -4,10 +4,10 @@
   <xacro:include filename="$(find drivebot_description)/urdf/macros.xacro" />
   <!-- X = front/back, Y = right/left, Z = up/down  -->
-  <xacro:property name="bodyX" value="0.6" />
-  <xacro:property name="bodyY" value="0.4" />
+  <xacro:property name="bodyX" value="0.9" />
+  <xacro:property name="bodyY" value="0.7" />
   <xacro:property name="bodyZ" value="0.2" />
   <xacro:property name="bodyMass" value="5" />
-  <xacro:property name="wheelR" value="${0.1 + 0.1}" />
-  <xacro:property name="wheelH" value="0.1" />
+  <xacro:property name="wheelR" value="${0.1}" />
+  <xacro:property name="wheelH" value="0.05" />
   <xacro:property name="wheelMass" value="1" />
   <xacro:property name="casterR" value="${(wheelR - bodyZ / 2) / 2}" />
@@ -24,33 +24,62 @@
   </gazebo>
   <xacro:cylinderLink
-      name="leftWheel" mass="${wheelMass}" radius="${wheelR}" height="${wheelH}" color="red" p ="${pi/2}" />
-  <joint name="leftWheel_joint" type="continuous">
+      name="leftRearWheel" mass="${wheelMass}" radius="${wheelR}" height="${wheelH}" color="red" p ="${pi/2}" />
+  <joint name="leftRearWheel_joint" type="continuous">
     <parent link="body_link" />
-    <child link="leftWheel_link" />
-    <origin xyz="${-bodyX/4} ${bodyY/2 + wheelH/2} 0" rpy="0 0 ${pi/2}" />
+    <child link="leftRearWheel_link" />
+    <origin xyz="${-bodyX/4} ${bodyY/2 + wheelH/2} ${-bodyZ/2}" rpy="0 0 ${pi/2}" />
   </joint>
-  <xacro:jointTransmission name="leftWheel" />
-  <gazebo reference="leftWheel_link">
+  <xacro:jointTransmission name="leftRearWheel" />
+  <gazebo reference="leftRearWheel_link">
     <material>Gazebo/Red</material>
+    <mu1 value="1.0"/>
+    <mu2 value="1.0"/>
+    <kp value="10000000.0" />
+    <kd value="1.0" />
   </gazebo>
   <xacro:cylinderLink
-      name="rightWheel" mass="${wheelMass}" radius="${wheelR}" height="${wheelH}" color="green" p ="${pi/2}"/>
-  <joint name="rightWheel_joint" type="continuous">
+      name="rightRearWheel" mass="${wheelMass}" radius="${wheelR}" height="${wheelH}" color="green" p ="${pi/2}"/>
+  <joint name="rightRearWheel_joint" type="continuous">
     <parent link="body_link" />
-    <child link="rightWheel_link" />
-    <origin xyz="${-bodyX/4} ${-bodyY/2 - wheelH/2} 0" rpy="0 0 ${pi/2}" />
+    <child link="rightRearWheel_link" />
+    <origin xyz="${-bodyX/4} ${-bodyY/2 - wheelH/2} ${-bodyZ/2}" rpy="0 0 ${pi/2}" />
   </joint>
-  <xacro:jointTransmission name="rightWheel" />
-  <gazebo reference="rightWheel_link">
+  <xacro:jointTransmission name="rightRearWheel" />
+  <gazebo reference="rightRearWheel_link">
     <material>Gazebo/Green</material>
+    <mu1 value="1.0"/>
+    <mu2 value="1.0"/>
+    <kp value="10000000.0" />
+    <kd value="1.0" />
   </gazebo>
-  <xacro:sphereLink name="caster" mass="${casterMass}" r="${casterR}" color="black" />
-  <joint name="caster_joint" type="fixed">
+  <xacro:cylinderLink
+      name="leftFrontWheel" mass="${wheelMass}" radius="${wheelR}" height="${wheelH}" color="red" p ="${pi/2}" />
+  <joint name="leftFrontWheel_joint" type="continuous">
     <parent link="body_link" />
-    <child link="caster_link" />
-    <origin xyz="${bodyX/4} 0 ${-(bodyZ/2 + casterR)}" rpy="0 0 0" />
+    <child link="leftFrontWheel_link" />
+    <origin xyz="${bodyX/4} ${bodyY/2 + wheelH/2} ${-bodyZ/2}" rpy="0 0 ${pi/2}" />
   </joint>
-  <gazebo reference="caster_link">
-    <material>Gazebo/Black</material>
+  <xacro:jointTransmission name="leftFrontWheel" />
+  <gazebo reference="leftFrontWheel_link">
+    <material>Gazebo/Red</material>
+    <mu1 value="1.0"/>
+    <mu2 value="1.0"/>
+    <kp value="10000000.0" />
+    <kd value="1.0" />
+  </gazebo>
+  <xacro:cylinderLink
+      name="rightFrontWheel" mass="${wheelMass}" radius="${wheelR}" height="${wheelH}" color="green" p ="${pi/2}"/>
+  <joint name="rightFrontWheel_joint" type="continuous">
+    <parent link="body_link" />
+    <child link="rightFrontWheel_link" />
+    <origin xyz="${bodyX/4} ${-bodyY/2 - wheelH/2} ${-bodyZ/2}" rpy="0 0 ${pi/2}" />
+  </joint>
+  <xacro:jointTransmission name="rightFrontWheel" />
+  <gazebo reference="rightFrontWheel_link">
+    <material>Gazebo/Green</material>
+    <mu1 value="1.0"/>
+    <mu2 value="1.0"/>
+    <kp value="10000000.0" />
+    <kd value="1.0" />
   </gazebo>
   <!-- ros_control plugin -->

File: drivebot_description/urdf/macros.xacro (robot description, xacro)
@@ -85,12 +85,11 @@
     </link>
   </xacro:macro>
-  <xacro:macro name="jointTransmission" params="name reduction:=10">
+  <xacro:macro name="jointTransmission" params="name reduction:=1">
     <transmission name="${name}_transmission">
       <type>transmission_interface/SimpleTransmission</type>
       <joint name="${name}_joint">
-        <hardwareInterface>hardware_interface/EffortJointInterface</hardwareInterface>
+        <hardwareInterface>hardware_interface/VelocityJointInterface</hardwareInterface>
       </joint>
       <actuator name="${name}_servo">
-        <hardwareInterface>EffortJointInterface</hardwareInterface>
         <mechanicalReduction>${reduction}</mechanicalReduction>
       </actuator>
